File: Prototype/40-KICAD/LED_Board/MCU_Board/MCU_Board.kicad_pcb (KiCad board)
At the start: 2 copper layers, 39 x 39 mm, 30 parts, among them J1 Conn_01x01, J10 Conn_01x01, J11 Conn_01x01, J12 Conn_01x01, J13 Conn_01x01, J16 Conn_01x04, J18 Conn_01x02, J19 Conn_01x02, J2 Conn_01x01, J20 Conn_01x04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

Commit message: 12V ws2815 compatibility
Parts:
- added C2: 1uF, Capacitor_SMD:C_0805_2012Metric_Pad1.18x1.45mm_HandSolder, F.Cu at (103.0, 111.6)
- added C3: 2.2uF, Capacitor_SMD:C_0805_2012Metric_Pad1.18x1.45mm_HandSolder, F.Cu at (97.1, 111.5)
- added Q1: 2N7000, Package_TO_SOT_SMD:SOT-23, F.Cu at (96.0, 85.8)
- added R8: 10K, Resistor_SMD:R_0603_1608Metric_Pad0.98x0.95mm_HandSolder, F.Cu at (98.5, 86.1)
- added R9: 10K, Resistor_SMD:R_0603_1608Metric_Pad0.98x0.95mm_HandSolder, F.Cu at (93.7, 83.9)
- added U3: MIC5219-5.0YM5, Package_TO_SOT_SMD:SOT-23-5, F.Cu at (100.5, 107.7)
- moved R3 3.32 mm to (96.3, 83.0), turned to 180 degrees
- moved J20 2.53 mm to (104.4, 86.7)
Connections:
- J18 pad 1: +5V -> +12V
- J18 pad 2: +5V -> +12V
- J19 pad 1: +5V -> +12V
- J19 pad 2: +5V -> +12V
- J2 pad 1: +5V -> +12V
- J8 pad 1: +5V -> +12V
- R3 pad 2: B0 -> NEOPIXEL
Routing:
- net +5V: track 31.0 -> 51.6 mm, vias 3 -> 4
- net +12V: track 0.00 -> 10.00 mm, vias 0 -> 1
- net NEOPIXEL: track 0.00 -> 3.83 mm
- net B0: track 7.07 -> 10.4 mm
- net Net-(J3-Pad1): track 5.83 -> 2.79 mm
- net B2: track 12.0 -> 13.6 mm
- added copper zone on B.Cu, net +12V
- removed copper zone on B.Cu, net +5V

Commit message: Updated PCB
Level shifter not required for ws2815 (5V logic)
Parts:
- removed Q1: 2N7000, Package_TO_SOT_SMD:SOT-23
- removed R8, R9: 10K, Resistor_SMD:R_0603_1608Metric_Pad0.98x0.95mm_HandSolder
- moved J20 2.50 mm to (101.9, 86.7)
- moved R3 1.57 mm to (96.4, 84.5), turned to -90 degrees
Connections:
- R3 pad 2: NEOPIXEL -> B0
Routing:
- net +5V: track 51.6 -> 45.2 mm, vias 4 -> 3
- net NEOPIXEL: track 3.83 -> 0.00 mm
- net B0: track 10.4 -> 8.08 mm
- net B2: track 13.6 -> 11.9 mm
- net Net-(J3-Pad1): track 2.79 -> 3.87 mm
- net +12V: track 10.00 -> 8.94 mm, vias 1 -> 0
