File: Prototype/40-KICAD/LED_Board/MCU_Board/MCU_Board.kicad_sch (KiCad schematic)
At the start: 34 parts, among them J1 Conn_01x01, J10 Conn_01x01, J11 Conn_01x01, J12 Conn_01x01, J13 Conn_01x01, J16 Conn_01x04, J17 Conn_01x04, J18 Conn_01x02, J19 Conn_01x02, J2 Conn_01x01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

Commit message: 12V ws2815 compatibility
Parts:
- added C2: 1uF, Capacitor_SMD:C_0805_2012Metric_Pad1.18x1.45mm_HandSolder, symbol Device:C
- added C3: 2.2uF, Capacitor_SMD:C_0805_2012Metric_Pad1.18x1.45mm_HandSolder, symbol Device:C
- added Q1: 2N7000, Package_TO_SOT_SMD:SOT-23, symbol Transistor_FET:2N7000
- added R8, R9: 10K, Resistor_SMD:R_0603_1608Metric_Pad0.98x0.95mm_HandSolder, symbol Device:R
- added U3: MIC5219-5.0YM5, Package_TO_SOT_SMD:SOT-23-5, symbol Regulator_Linear:MIC5219-5.0YM5
Connections:
- net +5V: now also C3.1, Q1.2 (G), R8.1, U3.5 (OUT); no longer J18.1 (Pin_1), J18.2 (Pin_2), J19.1 (Pin_1), J19.2 (Pin_2), J2.1 (Pin_1), J8.1 (Pin_1)
- net B0: now also Q1.1 (S), R8.2; no longer R3.2
- net GND: now also C2.2, C3.2, U3.2 (GND)
- new net +12V: C2.1, J18.1 (Pin_1), J18.2 (Pin_2), J19.1 (Pin_1), J19.2 (Pin_2), J2.1 (Pin_1), J8.1 (Pin_1), R9.1, U3.1 (IN)
- new net NEOPIXEL: Q1.3 (D), R3.2, R9.2

Commit message: Updated PCB
Level shifter not required for ws2815 (5V logic)
Parts:
- removed Q1: 2N7000, Package_TO_SOT_SMD:SOT-23, symbol Transistor_FET:2N7000
- removed R8, R9: 10K, Resistor_SMD:R_0603_1608Metric_Pad0.98x0.95mm_HandSolder, symbol Device:R
Connections:
- net NEOPIXEL is gone; now on net B0: R3.2
